File: HW2/PIC_breakout_pcb/ME433.brd (EAGLE design)
At the start: 50 x 50 mm, 24 parts

Commit message: add gerber file for pic breakout
Parts:
- removed LED1, LED2: (no value), SparkFun:LED3MM
- added A4, PWR: (no value), SparkFun:LED3MM
- C4: value 0.1uF -> 10uF
- JP1, JP2: device SparkFun:1X08_LONGPADS -> SparkFun:1X08
- moved JP1 22.6 mm to (1.27, 16.5), turned to 90 degrees
- moved JP2 22.1 mm to (48.8, 16.5), turned to 90 degrees
- moved C3 1.41 mm to (45.1, 16.7), turned to 270 degrees
- moved C9 0.56 mm to (34.2, 11.4)
- moved C2 0.50 mm to (31.3, 5.10)
- moved R1 0.25 mm to (8.23, 12.8)
- moved R2 0.25 mm to (11.2, 12.8)
- moved R4 0.25 mm to (4.96, 12.8)
- renumbered S1 to RESET, S2 to USER
Connections:
- net +3V3: now also JP1.2, PWR.A; no longer JP1.7, LED1.A
- net 5V: now also JP2.2; no longer JP2.7
- net GND: now also JP1.1, JP2.1; no longer JP1.8, JP2.8
- net N$12: now also PWR.K; no longer LED1.K
- net N$3: now also A4.K; no longer LED2.K
- net RA0: now also JP1.8; no longer JP1.1
- net RA1: now also JP1.7; no longer JP1.2
- net RA4: now also A4.A, JP1.3; no longer JP1.6, LED2.A
- net RB13: now also JP2.6; no longer JP2.3
- net RB14: now also JP2.7; no longer JP2.2
- net RB15: now also JP2.8; no longer JP2.1
- net RB2: now also JP1.6; no longer JP1.3
- net RB3: now also JP1.5; no longer JP1.4
- net RB4: now also JP1.4; no longer JP1.5
- net RB7: now also JP2.3; no longer JP2.6
- net RB8: now also JP2.4; no longer JP2.5
- net RB9: now also JP2.5; no longer JP2.4
Routing:
- net RA1: track 0.00 -> 24.3 mm
- net RA0: track 0.00 -> 24.3 mm
- net RA4: track 21.5 -> 44.1 mm
- net RB4: track 28.2 -> 50.4 mm
- net RB3: track 0.00 -> 22.2 mm
- net RB2: track 0.00 -> 22.2 mm
- net RB9: track 0.00 -> 21.9 mm
- net RB8: track 0.00 -> 21.9 mm
- net RB7: track 0.00 -> 21.9 mm
- net RB15: track 0.00 -> 20.7 mm
- net RB14: track 0.00 -> 20.7 mm
- net RB13: track 0.00 -> 20.7 mm
- net USB_ID: track 24.6 -> 22.0 mm
- net 5V: track 1.74 -> 0.00 mm
- net N$12: track 4.37 -> 3.62 mm
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Other:
- board text added: "3V3"
- board text added: "5V"
- board text added: "A0"
- board text added: "A1"
- board text added: "A4"
- board text added: "B13"
- board text added: "B14"
- board text added: "B15"
- board text added: "B2"
- board text added: "B3"
- board text added: "B4"
- board text added: "B7"
- board text added: "B8"
- board text added: "B9"
- board text added: "Francis Chen ME 433"
