File: HW2/PIC_breakout_pcb/ME433.sch (EAGLE design)
At the start: 24 parts

Commit message: add gerber file for pic breakout
Parts:
- C4: value 0.1uF -> 10uF
- JP1, JP2: device SparkFun:M08LONGPADS -> SparkFun:M08
- renumbered LED1 to PWR, LED2 to A4, S1 to RESET, S2 to USER
Connections:
- net +3V3: now also JP1.2; no longer JP1.7
- net 5V: now also JP2.2; no longer JP2.7
- net GND: now also JP1.1, JP2.1; no longer JP1.8, JP2.8
- net RA0: now also JP1.8; no longer JP1.1
- net RA1: now also JP1.7; no longer JP1.2
- net RA4: now also JP1.3; no longer JP1.6
- net RB13: now also JP2.6; no longer JP2.3
- net RB14: now also JP2.7; no longer JP2.2
- net RB15: now also JP2.8; no longer JP2.1
- net RB2: now also JP1.6; no longer JP1.3
- net RB3: now also JP1.5; no longer JP1.4
- net RB4: now also JP1.4; no longer JP1.5
- net RB7: now also JP2.3; no longer JP2.6
- net RB8: now also JP2.4; no longer JP2.5
- net RB9: now also JP2.5; no longer JP2.4
Other:
- moved on the sheet: JP1, JP2
